File: boards/driver/driverboard.kicad_pcb (KiCad board)
At the start: 2 copper layers, 49.5 x 54.6 mm, 44 parts, among them J1 RJ45, J2 RJ45, P1 HE10-10, Q1 NDS355, Q2 NDS355, Q3 NDS355, Q4 NDS355, Q5 NDS355, Q6 NDS355, Q7 NDS355, Q8 NDS355, U1 74HC595, U2 TS2937

Commit message: Final version 1.0
Changed lines of the file:
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@@
       (plotinvisibletext false)
       (padsonsilk false)
-      (subtractmaskfromsilk false)
+      (subtractmaskfromsilk true)
       (outputformat 1)
       (mirror false)
       (drillshape 0)
       (scaleselection 1)
-      (outputdirectory plot/))
+      (outputdirectory gerber/))
   )
   (net 0 "")
@@
     (fp_line (start -7.9375 5.0165) (end 7.9375 5.0165) (layer F.SilkS) (width 0.127))
     (fp_line (start 7.9375 -10.7315) (end -7.9375 -10.7315) (layer F.SilkS) (width 0.127))
-    (pad "" np_thru_hole circle (at 5.715 0) (size 3 3) (drill 3)
-      (layers *.Cu *.SilkS *.Mask)
-    )
-    (pad "" np_thru_hole circle (at -5.715 0) (size 3 3) (drill 3)
-      (layers *.Cu *.SilkS *.Mask)
+    (pad "" thru_hole circle (at 5.715 0) (size 3 3) (drill 3)
+      (layers *.Cu *.Mask F.SilkS)
+    )
+    (pad "" thru_hole circle (at -5.715 0) (size 3 3) (drill 3)
+      (layers *.Cu *.Mask F.SilkS)
     )
     (pad 1 thru_hole rect (at -4.445 -6.35) (size 1.50114 1.50114) (drill 0.89916)
@@
     (fp_line (start -7.9375 5.0165) (end 7.9375 5.0165) (layer F.SilkS) (width 0.127))
     (fp_line (start -7.9375 -10.7315) (end 7.9375 -10.7315) (layer F.SilkS) (width 0.127))
-    (pad "" np_thru_hole circle (at 5.715 0) (size 3 3) (drill 3)
-      (layers *.Cu *.SilkS *.Mask)
-    )
-    (pad "" np_thru_hole circle (at -5.715 0) (size 3 3) (drill 3)
-      (layers *.Cu *.SilkS *.Mask)
+    (pad "" thru_hole circle (at 5.715 0) (size 3 3) (drill 3)
+      (layers *.Cu *.Mask F.SilkS)
+    )
+    (pad "" thru_hole circle (at -5.715 0) (size 3 3) (drill 3)
+      (layers *.Cu *.Mask F.SilkS)
     )
     (pad 1 thru_hole rect (at -4.445 -6.35) (size 1.50114 1.50114) (drill 0.89916)
@@
   (segment (start 123.825 54.61) (end 120.015 54.61) (width 1) (layer B.Cu) (net 1))
   (segment (start 120.015 54.61) (end 116.205 54.61) (width 1) (layer B.Cu) (net 1))
-  (segment (start 107.315 40.767) (end 107.315 41.91) (width 0.5) (layer F.Cu) (net 2) (status 400000))
+  (segment (start 107.315 40.767) (end 107.315 41.91) (width 0.5) (layer F.Cu) (net 2))
   (via (at 107.315 41.91) (size 0.6) (drill 0.2) (layers F.Cu B.Cu) (net 2))
   (segment (start 107.315 41.91) (end 108.585 43.18) (width 0.5) (layer B.Cu) (net 2))
