File: boards/panelized/panelized.kicad_pcb (KiCad board)
At the start: 2 copper layers, 99.7 x 54.6 mm, 88 parts, among them J1 RJ45, J2 RJ45, P1 HE10-10, Q1 NDS355, Q2 NDS355, Q3 NDS355, Q4 NDS355, Q5 NDS355, Q6 NDS355, Q7 NDS355, Q8 NDS355, U1 74HC595, U2 TS2937

Commit message: Final version 1.0
Parts:
- removed the 1PIN at (96.8, 36.6)
- removed the 1PIN at (96.8, 86.6)
- removed the 1PIN at (51.8, 86.6)
- removed the 1PIN at (51.8, 36.6)
- removed the C1 at (85.1, 67.9)
- removed the C2 at (55.2, 63.5)
- removed the C3 at (51.4, 55.2)
- removed the C4 at (61.6, 63.5)
- removed the C5 at (61.6, 55.2)
- removed the D1 at (55.2, 36.2)
- removed the D2 at (57.1, 57.1)
- removed the D3 at (57.1, 36.2)
- removed the G*** at (79.4, 48.1)
- removed the J1 at (64.1, 81.9)
- removed the P1 at (74.3, 38.7)
- removed the Q1 at (92.7, 52.1)
- removed the Q2 at (88.9, 52.1)
- removed the R1 at (55.2, 40.0)
- removed the R10 at (67.9, 54.6)
- removed the R11 at (92.1, 47.0)
- removed the R12 at (88.3, 47.0)
- removed the R2 at (57.1, 40.0)
- removed the R3 at (94.6, 54.6)
- removed the R4 at (90.8, 54.6)
- removed the R5 at (87.0, 54.6)
- removed the R6 at (83.2, 54.6)
- removed the R7 at (79.4, 54.6)
- removed the R8 at (75.6, 54.6)
- removed the R9 at (71.8, 54.6)
- removed the U1 at (78.7, 64.1)
- removed the U2 at (56.5, 53.3)
- added 1PIN: P***, 1pin, F.Cu at (146.9, 36.6)
- added 1PIN: P***, 1pin, F.Cu at (128.3, 94.0)
- added 1PIN: P***, 1pin, F.Cu at (128.3, 129.5)
- added 1PIN: P***, 1pin, F.Cu at (53.3, 129.5)
- added 1PIN: P***, 1pin, F.Cu at (146.9, 86.6)
- added 1PIN: P***, 1pin, F.Cu at (102.0, 86.6)
- added 1PIN: P***, 1pin, F.Cu at (102.0, 36.6)
- added 1PIN: P***, 1pin, F.Cu at (53.3, 94.0)
- added C1: 100n, SM0603, F.Cu at (135.3, 67.9)
- added C1: 100n, SM0603, F.Cu at (101.0, 116.8)
- added C2: 10uF, c_tant_D, F.Cu at (105.4, 63.5)
- added C2: 100nf, SM0603, F.Cu at (89.5, 120.0)
- added C3: 100nF, SM0603, F.Cu at (101.6, 55.2)
- added C3: 10uF, c_tant_D, F.Cu at (90.8, 100.3)
- added C4: 10uF, c_tant_D, F.Cu at (111.8, 63.5)
- added C4: 100nF, SM0603, F.Cu at (111.1, 94.6)
- added C5: 100nF, SM0603, F.Cu at (111.8, 55.2)
- added C5: 10uF, c_tant_D, F.Cu at (99.1, 102.9)
- added C6: 100nF, SM0603, F.Cu at (111.1, 105.4)
- added C7: 100nf, SM0603, F.Cu at (107.3, 121.3)
- added D1: LED, SM0603, F.Cu at (105.4, 36.2)
- added D1: LED, SM0603, F.Cu at (121.9, 109.2)
- added D2: BAT42W, sod123, F.Cu at (107.3, 57.1)
- added D2: LED, SM0603, F.Cu at (121.9, 107.3)
- added D3: LED, SM0603, F.Cu at (107.3, 36.2)
- added D3: BAT42W, sod123, F.Cu at (108.0, 100.3)
- added D4: LED, SM0603, F.Cu at (121.9, 105.4)
- added F1: FUSE, fuse1, F.Cu at (75.6, 101.6)
- added G***: logo_silkbot_30_00mm, logo_silkbot_30_00mm, B.Cu at (129.5, 48.1)
- added G***: logo_silkbot_30_00mm, logo_silkbot_30_00mm, B.Cu at (107.3, 100.3)
- added J1: RJ45, RJ45_MEBP_8-8G, F.Cu at (64.1, 82.5)
- added J1: RJ45, RJ45_MEBP_8-8G, F.Cu at (60.3, 113.7)
- added P1: HE10-10, HE10-10C, F.Cu at (124.5, 38.7)
- added P1: CONN_2, bornier2, F.Cu at (69.2, 94.0)
- added P2: CONN_7, SIL-7, F.Cu at (83.8, 127.0)
- added Q1: NDS355, sot23, F.Cu at (142.9, 52.1)
- added Q1: IRLR110, DPAK2, F.Cu at (113.7, 127.0)
- added Q2: NDS355, sot23, F.Cu at (139.1, 52.1)
- added Q2: NDS355, sot23, F.Cu at (89.5, 123.2)
- added R1: 1k, SM0603, F.Cu at (105.4, 40.0)
- added R1: 10k, SM0603, F.Cu at (94.6, 108.6)
- added R10: 200, SM0603, F.Cu at (118.1, 54.6)
- added R10: 1k, SM0603, F.Cu at (118.7, 105.4)
- added R11: 160, SM1206, F.Cu at (142.2, 47.0)
- added R11: 1k, SM0603, F.Cu at (87.6, 120.0)
- added R12: 160, SM1206, F.Cu at (138.4, 47.0)
- added R12: 1k, SM0603, F.Cu at (86.4, 129.5)
- added R2: 1k, SM0603, F.Cu at (107.3, 40.0)
- added R2: 90k, SM0603, F.Cu at (98.4, 108.6)
- added R3: 200, SM0603, F.Cu at (144.8, 54.6)
- added R3: 1k, SM0603, F.Cu at (109.9, 121.3)
- added R4: 200, SM0603, F.Cu at (141.0, 54.6)
- added R4: 100k, SM0603, F.Cu at (101.0, 113.7)
- added R5: 200, SM0603, F.Cu at (137.2, 54.6)
- added R5: 0.05, SM1206, F.Cu at (69.2, 127.0)
- added R6: 200, SM0603, F.Cu at (133.3, 54.6)
- added R6: 1k, SM0603, F.Cu at (98.4, 120.0)
- added R7: 200, SM0603, F.Cu at (129.5, 54.6)
- added R7: 1k, SM0603, F.Cu at (118.7, 109.2)
- added R8: 200, SM0603, F.Cu at (125.7, 54.6)
- added R8: 1k, SM0603, F.Cu at (105.4, 121.3)
- added R9: 200, SM0603, F.Cu at (121.9, 54.6)
- added R9: 1k, SM0603, F.Cu at (118.7, 107.3)
- added RV1: POT, trimmer_piher_pt6xh, F.Cu at (99.1, 125.7)
- added SW1: SW_PUSH, SW_PUSH_SMALL, F.Cu at (120.0, 118.1)
- added U1: 74HC595, SO16E, F.Cu at (128.9, 64.1)
- added U1: LM358, SO8E, F.Cu at (96.5, 113.7)
- added U2: TS2937, DPAK2, F.Cu at (106.7, 53.3)
- added U2: SN74LVC1G74, SO8E, F.Cu at (105.4, 113.7)
- added U3: 74HCT125, SO14E, F.Cu at (85.1, 113.7)
- added U4: TS2937, DPAK2, F.Cu at (113.7, 100.3)
- moved C4 50.2 mm to (61.6, 63.5)
- moved C5 50.2 mm to (61.6, 55.2)
- moved Q1 50.2 mm to (92.7, 52.1)
- moved Q5 50.2 mm to (127.6, 52.1)
- moved Q5 50.2 mm to (77.5, 52.1)
- moved Q6 50.2 mm to (123.8, 52.1)
- moved Q6 50.2 mm to (73.7, 52.1)
- moved Q7 50.2 mm to (120.0, 52.1)
- moved Q7 50.2 mm to (69.8, 52.1)
- moved R10 50.2 mm to (67.9, 54.6)
- moved R11 50.2 mm to (92.1, 47.0)
- moved R12 50.2 mm to (88.3, 47.0)
- moved R13 50.2 mm to (134.6, 47.0)
- moved R13 50.2 mm to (84.5, 47.0)
- moved R14 50.2 mm to (130.8, 47.0)
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Routing:
- net +24V: track 254.5 -> 364.5 mm, vias 22 -> 24
- net +5V: track 115.5 -> 202.0 mm, vias 4 -> 9
- net Sense: track 0.00 -> 67.1 mm, vias 0 -> 1
- net N-0000027: track 0.00 -> 65.2 mm
- net BusOff: track 0.00 -> 63.9 mm, vias 0 -> 6
- net N-0000024: track 6.46 -> 33.3 mm, vias 0 -> 1
- net PowerOn: track 0.00 -> 26.2 mm
- net 3.3_Clock: track 0.00 -> 25.0 mm, vias 0 -> 2
- net Clock: track 68.7 -> 92.5 mm
- net 3.3_Enable: track 0.00 -> 23.7 mm, vias 0 -> 4
- net Reset: track 66.9 -> 87.3 mm, vias 2 -> 3
- net Data_Out: track 68.1 -> 87.2 mm, vias 4 -> 7
- net Enable: track 74.6 -> 93.2 mm, vias 4 -> 5
- net Shutdown: track 0.00 -> 16.8 mm, vias 0 -> 2
- net N-0000012: track 0.00 -> 13.2 mm
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Other:
- board size 99.7 x 54.6 mm -> 99.7 x 99.1 mm
- board text added: "+3.3V"
- board text added: "BOFF"
- board text added: "CLK"
- board text added: "DO"
- board text added: "EN"
- board text added: "GND"
- board text added: "Levelshifter"
- board text added: "RST"
- board text added: "https://github.com/LongHairedHacker/HeptaLED"
